File: m4pyro/m4pyro.kicad_pcb (KiCad board)
At the start: 2 copper layers, 100 x 75 mm, 162 parts, among them IC1 STM32F405RxTx, IC10 LTC4151, IC2 TPS62133, IC3 MCP2562, IC4 TPS62153, IC5 ADP2389, IC6 LTC4151, IC7 ADP2389, IC8 LTC4151, IC9 ADP2389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

Commit message: added gnd vias and continuity circuits
Parts:
- moved D14 37.1 mm to (78.7, 140.6), turned to 270 degrees
- moved C50 35.7 mm to (77.0, 140.6), turned to 270 degrees
- moved R60 32.1 mm to (80.4, 139.7), turned to 90 degrees
- moved R63 31.7 mm to (80.4, 141.8), turned to 270 degrees
- moved C49 19.4 mm to (89.6, 145.2), turned to 90 degrees
- moved D13 17.9 mm to (87.0, 144.2)
- moved R58 17.8 mm to (84.1, 139.6), turned to 90 degrees
- moved R62 17.5 mm to (88.0, 145.8)
- moved R59 15.2 mm to (85.8, 145.8), turned to 180 degrees
- moved R61 14.6 mm to (84.1, 141.8), turned to 270 degrees
- moved D12 13.9 mm to (82.4, 141.2), turned to 270 degrees
- moved C48 12.5 mm to (84.2, 144.0), turned to 90 degrees
Routing:
- net GND: track 108.6 -> 205.0 mm, vias 16 -> 130
- net /VALVE_3: track 38.6 -> 71.0 mm
- net /V2_CONT: track 0.00 -> 18.2 mm, vias 0 -> 2
- net /VALVE_2: track 12.8 -> 31.0 mm
- net 3v3: track 16.3 -> 32.3 mm
- net /V1_CONT: track 0.00 -> 13.6 mm, vias 0 -> 2
- net /VALVE_1: track 11.7 -> 23.3 mm
- net /V3_CONT: track 0.00 -> 6.22 mm

Commit message: started mcu layout
Parts:
- moved C1 217.9 mm to (72.0, 106.1), turned to 90 degrees
- moved R1 201.7 mm to (76.0, 106.1), turned to 90 degrees
- moved C2 197.2 mm to (74.0, 108.3)
- moved Y1 159.7 mm to (74.0, 106.1)
- moved IC3 148.0 mm to (64.7, 105.7), turned to 180 degrees
- moved IC1 140.1 mm to (77.1, 96.3), turned to 90 degrees
Connections:
- IC1 pad 42: /UART_TX -> (no net)
- IC1 pad 43: /UART_RX -> (no net)
- IC1 pad 58: (no net) -> /UART_TX
- IC1 pad 59: (no net) -> /UART_RX
Routing:
- net /SDA: track 0.00 -> 99.4 mm, vias 0 -> 5
- net /SCL: track 0.00 -> 99.3 mm, vias 0 -> 5
- net 3v3: track 32.3 -> 88.1 mm
- net /V1_CONT: track 13.6 -> 67.3 mm
- net /V3_CONT: track 6.22 -> 59.3 mm
- net /V2_CONT: track 18.2 -> 71.1 mm
- net /V3_FIRE: track 0.00 -> 49.9 mm, vias 0 -> 3
- net /V2_FIRE: track 0.00 -> 31.9 mm, vias 0 -> 3
- net /JTMS: track 3.22 -> 18.9 mm
- net /JTDO: track 0.00 -> 12.8 mm, vias 0 -> 1
- net GND: track 205.0 -> 217.2 mm, vias 130 -> 138
- net /CAN_TXD: track 0.00 -> 12.1 mm
- net /JTDI: track 1.47 -> 13.5 mm, vias 1 -> 0
- net /UART_RX: track 3.32 -> 15.0 mm
- net /JTCK: track 3.28 -> 15.0 mm
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
Commit message: pcb progress
Parts:
- moved C4 205.1 mm to (72.9, 88.2), turned to 270 degrees
- moved C7 202.1 mm to (69.4, 106.1), turned to 90 degrees
- moved C3 193.5 mm to (70.7, 106.1), turned to 90 degrees
- moved C9 187.8 mm to (85.3, 92.1), turned to 180 degrees
- moved C5 187.7 mm to (69.4, 101.5), turned to 90 degrees
- moved C15 182.9 mm to (64.5, 102.9)
- moved C11 182.1 mm to (74.1, 88.2), turned to 90 degrees
- moved C18 181.2 mm to (85.3, 93.3)
- moved C10 178.6 mm to (85.3, 99.1), turned to 180 degrees
- moved C6 156.0 mm to (79.3, 104.8), turned to 90 degrees
Routing:
- net 3v3: track 88.1 -> 155.3 mm, vias 2 -> 6
- net GND: track 217.2 -> 235.8 mm, vias 138 -> 154
- net /V1_FIRE: track 8.29 -> 16.4 mm, vias 1 -> 2
- net /V2_FIRE: track 31.9 -> 38.4 mm, vias 3 -> 4
- net /V3_FIRE: track 49.9 -> 56.1 mm, vias 3 -> 4
- net Net-(C18-Pad1): track 0.00 -> 2.15 mm
- net Net-(C11-Pad1): track 0.00 -> 2.05 mm
- net /~RST: track 0.00 -> 1.45 mm, vias 0 -> 1
- net /5v_CAN: track 12.2 -> 13.1 mm, vias 2 -> 3
