File: m4pyro/m4pyro.sch (KiCad schematic (older format))
At the start: 99 parts, among them IC1 STM32F405RxTx, IC2 TPS62133, IC3 MCP2562, IC4 TPS62153, J1 WEST TOP, J2 WEST BOT, J3 EAST TOP, J4 EAST BOT, P1 SWD_TC, Q1 Si5515CDC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

Commit message: added valve fire and monitor stuff, need to think about continuity
Parts:
- added C27, C34, C41: 10µ, agg:1206, symbol agg-kicad1:C
- added C28, C35, C42: 1µ, agg:0402, symbol agg-kicad:C
- added C29, C36, C43: 100n, agg:0402, symbol agg-kicad1:C
- added C30, C37, C44: 100n, agg:0603, symbol agg-kicad1:C
- added C31, C38, C45: 22n, agg:0402, symbol agg-kicad1:C
- added C32, C39, C46: 1.2u, agg:0805, symbol agg-kicad1:C
- added C33, C40, C47: 100µ, agg:1210, symbol agg-kicad1:C
- added IC10, IC6, IC8: LTC4151, agg:DFN-10-EP-LT, symbol agg-kicad1:LTC4151
- added IC5, IC7, IC9: ADP2389, agg:ADP2389ACPZ-R7, symbol agg-kicad2:ADP2389
- added L3, L4, L5: 2µ2, agg:WE-HCC-1090, symbol agg-kicad1:L
- added R41, R42: 4k7, agg:0402, symbol agg-kicad1:R
- added R43, R48, R53: 100k, agg:0402, symbol agg-kicad1:R
- added R44, R49, R54: 68k, agg:0603, symbol agg-kicad1:R
- added R45, R50, R55: 47.5k, agg:0603, symbol agg-kicad1:R
- added R46, R51, R56: 2.5k, agg:0603, symbol agg-kicad1:R
- added R47, R52, R57: 5m, agg:1206, symbol agg-kicad1:R
- C12: footprint agg:0603 -> agg:1206; Farnell 2211164 -> 2094044
- C13: footprint agg:0402 -> agg:0603; Farnell 2496771 -> 1740614
- C14: value 100n -> 10µ; footprint agg:0402 -> agg:1206; Farnell 2496771 -> 2094044
- C17: value 10µ -> 100n; Farnell 2211164 -> 1740614
- X1: value BACKUP 22µ -> BKUP 22µ
- gave numbers to parts that had none: 1
Connections:
- net labels added: SCL, SDA, V1_FIRE, V2_FIRE, V3_FIRE, V_1_SUPPLY, V_2_SUPPLY, V_3_SUPPLY
- wire segments 637 -> 973
- no-connect marks 7 -> 19
Other:
- note added: "12v @ 12A Max."
- note added: "Address: 0x67"
- note added: "Address: 0x69"
- note added: "Address: 0x6F"
- note added: "Consider valve continuity?"
- note added: "Fixed 5v Output"
- note added: "PYRO CHANNELS - Firing & Continuity"
- note added: "VALVE CHANNELS - Firing & Current Monitoring"
- note removed: "FIRING CHANNELS"

Commit message: pyro schematic almost done
Parts:
- added C48, C49, C50: 100n, agg:0402, symbol agg-kicad1:C
- added D12, D13, D14: PMEG3005AEA, agg:SOD-323, symbol agg-kicad1:SCHOTTKY
- added R58, R59, R60: 1k, agg:0402, symbol agg-kicad1:R
- added R61, R62, R63: 10k, agg:0402, symbol agg-kicad1:R
- J1, J3: footprint (none) -> agg:TFML-115-02-L-D-LC
- J2, J4: footprint (none) -> agg:SFML-115-02-L-D
Connections:
- net labels added: V1_CONT, V2_CONT, V3_CONT
- wire segments 973 -> 1025
- no-connect marks 19 -> 28
Other:
- note added: "Valve 1"
- note added: "Valve 2"
- note added: "Valve 3"
- note removed: "Consider valve continuity?"

Commit message: started pyro pcb
Parts:
- added X2, X3, X4, X5: HOLE, agg:M3_MOUNT, symbol agg-kicad:PART
- L3, L4, L5: footprint agg:WE-HCC-1090 -> agg:WE-HCC-1090
Changed lines of the file:
@@
 F 0 "L3" H 2800 1250 50  0000 C CNN
 F 1 "2µ2" H 2800 1150 50  0000 C CNN
-F 2 "agg:WE-HCC-1090 " H 2750 1200 50  0001 C CNN
+F 2 "agg:WE-HCC-1090" H 2750 1200 50  0001 C CNN
 F 3 "" H 2750 1200 50  0001 C CNN
 F 4 "1848248" H 2750 1200 60  0001 C CNN "Farnell"
@@
 F 0 "L4" H 6200 1250 50  0000 C CNN
 F 1 "2µ2" H 6200 1150 50  0000 C CNN
-F 2 "agg:WE-HCC-1090 " H 6150 1200 50  0001 C CNN
+F 2 "agg:WE-HCC-1090" H 6150 1200 50  0001 C CNN
 F 3 "" H 6150 1200 50  0001 C CNN
 F 4 "1848248" H 6150 1200 60  0001 C CNN "Farnell"
@@
 F 0 "L5" H 9600 1250 50  0000 C CNN
 F 1 "2µ2" H 9600 1150 50  0000 C CNN
-F 2 "agg:WE-HCC-1090 " H 9550 1200 50  0001 C CNN
+F 2 "agg:WE-HCC-1090" H 9550 1200 50  0001 C CNN
 F 3 "" H 9550 1200 50  0001 C CNN
 F 4 "1848248" H 9550 1200 60  0001 C CNN "Farnell"
@@
 Wire Wire Line
 	18100 8400 18200 8400
+$Comp
+L agg-kicad:PART X2
+U 1 1 5AA6A67C
+P 14350 9650
+F 0 "X2" H 14400 9750 50  0000 L CNN
+F 1 "HOLE" H 14400 9650 50  0000 L CNN
+F 2 "agg:M3_MOUNT" H 14350 9650 50  0001 C CNN
+F 3 "" H 14350 9650 50  0001 C CNN
+	1    14350 9650
+	1    0    0    -1
+$EndComp
+$Comp
+L agg-kicad:PART X3
+U 1 1 5AA6B102
+P 14350 9900
+F 0 "X3" H 14400 10000 50  0000 L CNN
+F 1 "HOLE" H 14400 9900 50  0000 L CNN
+F 2 "agg:M3_MOUNT" H 14350 9900 50  0001 C CNN
+F 3 "" H 14350 9900 50  0001 C CNN
+	1    14350 9900
+	1    0    0    -1
+$EndComp
+$Comp
+L agg-kicad:PART X4
+U 1 1 5AA6B29C
+P 14350 10150
+F 0 "X4" H 14400 10250 50  0000 L CNN
+F 1 "HOLE" H 14400 10150 50  0000 L CNN
+F 2 "agg:M3_MOUNT" H 14350 10150 50  0001 C CNN
+F 3 "" H 14350 10150 50  0001 C CNN
+	1    14350 10150
+	1    0    0    -1
+$EndComp
+$Comp
+L agg-kicad:PART X5
+U 1 1 5AA6B408
+P 14350 10400
+F 0 "X5" H 14400 10500 50  0000 L CNN
+F 1 "HOLE" H 14400 10400 50  0000 L CNN
+F 2 "agg:M3_MOUNT" H 14350 10400 50  0001 C CNN
+F 3 "" H 14350 10400 50  0001 C CNN
+	1    14350 10400
+	1    0    0    -1
+$EndComp
 $EndSCHEMATC

Commit message: laying out pyro valve components
Parts:
- added J6: VALVES, agg:ultra-fit-01x03, symbol agg-kicad:CONN_01x03
- J5: value PYRO -> SUPPLY; footprint (none) -> agg:ultra-fit-01x03; symbol agg-kicad:CONN_01x06 -> agg-kicad:CONN_01x03; Farnell (none) -> 2494347
Connections:
- wire segments 1025 -> 1026
- no-connect marks 28 -> 27
Other:
- note added: "MOLEX Conenctors"
- note removed: "MOLEX Conenctor"
Changed lines of the file:
@@
 UART_TX
 $Comp
-L agg-kicad:CONN_01x06 J5
+L agg-kicad:CONN_01x03 J5
 U 1 1 5D21ED89
-P 11500 6650
-F 0 "J5" H 11450 6750 50  0000 C CNN
-F 1 "PYRO" H 11500 6050 50  0000 C CNN
-F 2 "" H 11500 6650 50  0001 C CNN
-F 3 "" H 11500 6650 50  0001 C CNN
-	1    11500 6650
-	1    0    0    -1
-$EndComp
-Wire Wire Line
-	11600 6650 11700 6650
-Wire Wire Line
-	11600 6750 11700 6750
-Wire Wire Line
-	11600 6850 11700 6850
+P 11500 6400
+F 0 "J5" H 11450 6500 50  0000 C CNN
+F 1 "SUPPLY" H 11500 6100 50  0000 C CNN
+F 2 "agg:ultra-fit-01x03" H 11500 6400 50  0001 C CNN
+F 3 "" H 11500 6400 50  0001 C CNN
+F 4 "2494347" H 11500 6400 50  0001 C CNN "Farnell"
+	1    11500 6400
+	1    0    0    -1
+$EndComp
+Wire Wire Line
+	11600 6400 11700 6400
+Wire Wire Line
+	11600 6500 11700 6500
 Wire Wire Line
 	11600 6950 11700 6950
 Wire Wire Line
 	11600 7050 11700 7050
-Text Label 11700 6850 0    60   ~ 0
+Wire Wire Line
+	11600 7150 11700 7150
+Text Label 11700 6950 0    60   ~ 0
 VALVE_1
-Text Label 11700 6950 0    60   ~ 0
+Text Label 11700 7050 0    60   ~ 0
 VALVE_2
-Text Label 11700 7050 0    60   ~ 0
+Text Label 11700 7150 0    60   ~ 0
 VALVE_3
-Text Label 11700 6650 0    60   ~ 0
+Text Label 11700 6400 0    60   ~ 0
 PYRO_SI
-Text Label 11700 6750 0    60   ~ 0
+Text Label 11700 6500 0    60   ~ 0
 PYRO_SI
-NoConn ~ 11600 7150
-Wire Notes Line
-	11200 6400 12350 6400
 Text Notes 11250 7450 0    60   ~ 0
-MOLEX Conenctor
-Wire Notes Line
-	12350 6400 12350 7500
-Wire Notes Line
-	11200 6400 11200 7500
+MOLEX Conenctors
 Wire Notes Line
 	11200 7500 12350 7500
@@
 	1    0    0    -1
 $EndComp
+$Comp
+L agg-kicad:CONN_01x03 J6
+U 1 1 5A989F84
+P 11500 6950
+F 0 "J6" H 11450 7050 50  0000 C CNN
+F 1 "VALVES" H 11500 6650 50  0000 C CNN
+F 2 "agg:ultra-fit-01x03" H 11500 6950 50  0001 C CNN
+F 3 "" H 11500 6950 50  0001 C CNN
+F 4 "2494347" H 11500 6950 50  0001 C CNN "farnell"
+	1    11500 6950
+	1    0    0    -1
+$EndComp
+Wire Wire Line
+	11600 6600 11700 6600
+Text Label 11700 6600 0    60   ~ 0
+PYRO_SI
+Wire Notes Line
+	12350 6200 11200 6200
+Wire Notes Line
+	12350 6200 12350 7500
+Wire Notes Line
+	11200 6200 11200 7500
 $EndSCHEMATC

Commit message: started mcu layout
Parts:
- J5, J6: footprint agg:ultra-fit-01x03 -> agg:ULTRA-FIT-01x03
Changed lines of the file:
@@
 	3050 8650 3050 8700
 Wire Wire Line
-	13800 4300 13900 4300
-Wire Wire Line
 	13800 4500 13900 4500
 Wire Wire Line
@@
 Text Label 13800 4000 2    50   ~ 0
 CH8_CONT
-Text Label 13800 4300 2    50   ~ 0
+Text Label 15000 2000 0    50   ~ 0
 UART_RX
-Text Label 13800 4200 2    50   ~ 0
+Text Label 15000 1900 0    50   ~ 0
 UART_TX
 $Comp
@@
 F 0 "J5" H 11450 6500 50  0000 C CNN
 F 1 "SUPPLY" H 11500 6100 50  0000 C CNN
-F 2 "agg:ultra-fit-01x03" H 11500 6400 50  0001 C CNN
+F 2 "agg:ULTRA-FIT-01x03" H 11500 6400 50  0001 C CNN
 F 3 "" H 11500 6400 50  0001 C CNN
 F 4 "2494347" H 11500 6400 50  0001 C CNN "Farnell"
@@
 Wire Wire Line
 	13900 4400 13800 4400
-Wire Wire Line
-	13900 4200 13800 4200
 NoConn ~ 13900 4100
 NoConn ~ 14900 3900
@@
 	14900 2400 15000 2400
 NoConn ~ 14900 1800
-NoConn ~ 14900 1900
-NoConn ~ 14900 2000
 NoConn ~ 14900 1500
 NoConn ~ 14900 2700
@@
 F 0 "J6" H 11450 7050 50  0000 C CNN
 F 1 "VALVES" H 11500 6650 50  0000 C CNN
-F 2 "agg:ultra-fit-01x03" H 11500 6950 50  0001 C CNN
+F 2 "agg:ULTRA-FIT-01x03" H 11500 6950 50  0001 C CNN
 F 3 "" H 11500 6950 50  0001 C CNN
 F 4 "2494347" H 11500 6950 50  0001 C CNN "farnell"
@@
 Wire Notes Line
 	11200 6200 11200 7500
+NoConn ~ 13900 4200
+NoConn ~ 13900 4300
+Wire Wire Line
+	15000 1900 14900 1900
+Wire Wire Line
+	14900 2000 15000 2000
 $EndSCHEMATC

Commit message: made good progress on pyro routing
Changed lines of the file:
@@
 Text Label 15000 2100 0    60   ~ 0
 CAN_RXD
-Text Label 15000 4500 0    50   ~ 0
+Text Label 15000 3900 0    50   ~ 0
 LED_GRN
-Text Label 15000 4300 0    50   ~ 0
+Text Label 13800 4200 2    50   ~ 0
 LED_RED
-Text Label 15000 4400 0    50   ~ 0
+Text Label 13800 4100 2    50   ~ 0
 LED_YLW
 Wire Wire Line
@@
 Text Notes 10850 5500 0    60   ~ 0
 Voltage Monitoring
-Text Label 15000 2600 0    50   ~ 0
+Text Label 15000 2500 0    59   ~ 0
 CH5
-Text Label 15000 3600 0    50   ~ 0
+Text Label 15000 3500 0    59   ~ 0
 CH6
-Text Label 15000 3800 0    50   ~ 0
+Text Label 15000 1500 0    59   ~ 0
 CH7
-Text Label 15000 3500 0    50   ~ 0
+Text Label 15000 3400 0    59   ~ 0
 CH8
-Text Label 15000 2500 0    50   ~ 0
+Text Label 15000 3600 0    59   ~ 0
 CH1
-Text Label 15000 2800 0    50   ~ 0
+Text Label 15000 2800 0    59   ~ 0
 CH2
-Text Label 15000 3700 0    50   ~ 0
+Text Label 15000 2700 0    59   ~ 0
 CH3
-Text Label 15000 3400 0    50   ~ 0
+Text Label 15000 2600 0    59   ~ 0
 CH4
 Wire Notes Line
@@
 	15000 2800 14900 2800
 Wire Wire Line
-	14900 3600 15000 3600
-Wire Wire Line
 	15000 2500 14900 2500
 Wire Wire Line
 	14900 2600 15000 2600
-Wire Wire Line
-	15000 3700 14900 3700
-Wire Wire Line
-	14900 3800 15000 3800
 $Comp
 L agg-kicad1:PWR #FLG04
@@
 Wire Notes Line
 	10800 6000 10800 10400
-Text Label 13800 3300 2    50   ~ 0
+Text Label 13800 3700 2    50   ~ 0
 CH1_CONT
-Text Label 13800 3400 2    50   ~ 0
+Text Label 13800 3800 2    50   ~ 0
 CH2_CONT
-Text Label 13800 3500 2    50   ~ 0
+Text Label 13800 3900 2    50   ~ 0
 CH3_CONT
-Text Label 13800 3600 2    50   ~ 0
+Text Label 13800 4000 2    50   ~ 0
 CH4_CONT
-Text Label 13800 3700 2    50   ~ 0
+Text Label 13800 3600 2    50   ~ 0
 CH5_CONT
-Text Label 13800 3800 2    50   ~ 0
+Text Label 13800 3500 2    50   ~ 0
 CH6_CONT
-Text Label 13800 3900 2    50   ~ 0
+Text Label 13800 3400 2    50   ~ 0
 CH7_CONT
-Text Label 13800 4000 2    50   ~ 0
+Text Label 13800 3300 2    50   ~ 0
 CH8_CONT
 Text Label 15000 2000 0    50   ~ 0
@@
 	14900 4200 15000 4200
 Wire Wire Line
-	14900 4300 15000 4300
+	13900 4200 13800 4200
 Wire Wire Line
-	14900 4400 15000 4400
+	13900 4100 13800 4100
 Wire Wire Line
-	14900 4500 15000 4500
+	14900 3900 15000 3900
 Wire Wire Line
 	13900 4400 13800 4400
-NoConn ~ 13900 4100
-NoConn ~ 14900 3900
 NoConn ~ 14900 4700
 NoConn ~ 14900 3300
@@
 	14900 2400 15000 2400
 NoConn ~ 14900 1800
-NoConn ~ 14900 1500
-NoConn ~ 14900 2700
 $Comp
 L agg-kicad:PWR #FLG07
@@
 Wire Notes Line
 	11200 6200 11200 7500
-NoConn ~ 13900 4200
 NoConn ~ 13900 4300
 Wire Wire Line
@@
 Wire Wire Line
 	14900 2000 15000 2000
+Wire Wire Line
+	14900 1500 15000 1500
+NoConn ~ 14900 3800
+NoConn ~ 14900 3700
+Wire Wire Line
+	14900 2700 15000 2700
+Wire Wire Line
+	14900 3600 15000 3600
+NoConn ~ 14900 4300
+NoConn ~ 14900 4400
+NoConn ~ 14900 4500
 $EndSCHEMATC

Commit message: routed pyro board
Changed lines of the file:
@@
 Text Label 15000 2100 0    60   ~ 0
 CAN_RXD
+Text Label 13800 4200 2    50   ~ 0
+LED_GRN
 Text Label 15000 3900 0    50   ~ 0
-LED_GRN
-Text Label 13800 4200 2    50   ~ 0
 LED_RED
 Text Label 13800 4100 2    50   ~ 0
@@
 Text Label 11350 4850 2    50   ~ 0
 SI_DIV
+Text Label 15000 1400 0    50   ~ 0
+SI_DIV
 Text Label 15000 1300 0    50   ~ 0
-SI_DIV
-Text Label 15000 1400 0    50   ~ 0
 BUS_DIV
+Text Label 13800 4400 2    50   ~ 0
+3A_EN
 Text Label 13800 4500 2    50   ~ 0
-3A_EN
-Text Label 13800 4400 2    50   ~ 0
 1A_EN
 $Comp

Commit message: added ilim resistor to pyro board
Parts:
- added R64, R65, R66: 82.5k, agg:0402, symbol agg-kicad1:R
Connections:
- wire segments 1026 -> 1035
- no-connect marks 27 -> 24
Other:
- note added: "12v @ 8A Max."
- note removed: "12v @ 12A Max."
Changed lines of the file:
@@
 V1_FIRE
 NoConn ~ 1650 2100
-NoConn ~ 1650 2200
 $Comp
 L agg-kicad1:R R43
@@
 	2650 1200 2750 1200
 Text Notes 1700 3650 0    60   ~ 0
-12v @ 12A Max.
+12v @ 8A Max.
 Wire Wire Line
 	5850 2000 5950 2000
@@
 V2_FIRE
 NoConn ~ 5050 2100
-NoConn ~ 5050 2200
 $Comp
 L agg-kicad1:R R48
@@
 Wire Wire Line
 	6050 1200 6150 1200
-Text Notes 5100 3650 0    60   ~ 0
-12v @ 12A Max.
 Wire Wire Line
 	9250 2000 9350 2000
@@
 V3_FIRE
 NoConn ~ 8450 2100
-NoConn ~ 8450 2200
 $Comp
 L agg-kicad1:R R53
@@
 Wire Wire Line
 	9450 1200 9550 1200
-Text Notes 8500 3650 0    60   ~ 0
-12v @ 12A Max.
 Text Notes 550  700  0    98   ~ 20
 VALVE CHANNELS - Firing & Current Monitoring
@@
 NoConn ~ 14900 4400
 NoConn ~ 14900 4500
+$Comp
+L agg-kicad1:R R64
+U 1 1 5AABCF7D
+P 850 2650
+F 0 "R64" H 900 2700 50  0000 C CNN
+F 1 "82.5k" H 900 2600 50  0000 C CNN
+F 2 "agg:0402" H 850 2650 50  0001 C CNN
+F 3 "" H 850 2650 50  0001 C CNN
+F 4 "2694663" H -6600 1750 60  0001 C CNN "Farnell"
+	1    850  2650
+	0    -1   -1   0
+$EndComp
+Wire Wire Line
+	850  2550 850  2200
+Wire Wire Line
+	850  2200 1650 2200
+$Comp
+L agg-kicad1:GND #PWR0120
+U 1 1 5ABE9834
+P 850 2750
+F 0 "#PWR0120" H 720 2790 50  0001 L CNN
+F 1 "GND" H 850 2650 50  0000 C CNN
+F 2 "" H 850 2750 60  0000 C CNN
+F 3 "" H 850 2750 60  0000 C CNN
+	1    850  2750
+	1    0    0    -1
+$EndComp
+Wire Wire Line
+	850  2750 850  2650
+$Comp
+L agg-kicad1:R R65
+U 1 1 5AD16B02
+P 4250 2650
+F 0 "R65" H 4300 2700 50  0000 C CNN
+F 1 "82.5k" H 4300 2600 50  0000 C CNN
+F 2 "agg:0402" H 4250 2650 50  0001 C CNN
+F 3 "" H 4250 2650 50  0001 C CNN
+F 4 "2694663" H -3200 1750 60  0001 C CNN "Farnell"
+	1    4250 2650
+	0    -1   -1   0
+$EndComp
+Wire Wire Line
+	4250 2550 4250 2200
+Wire Wire Line
+	4250 2200 5050 2200
+$Comp
+L agg-kicad1:GND #PWR0121
+U 1 1 5AD16B0A
+P 4250 2750
+F 0 "#PWR0121" H 4120 2790 50  0001 L CNN
+F 1 "GND" H 4250 2650 50  0000 C CNN
+F 2 "" H 4250 2750 60  0000 C CNN
+F 3 "" H 4250 2750 60  0000 C CNN
+	1    4250 2750
+	1    0    0    -1
+$EndComp
+Wire Wire Line
+	4250 2750 4250 2650
+$Comp
+L agg-kicad1:R R66
+U 1 1 5AE46060
+P 7650 2650
+F 0 "R66" H 7700 2700 50  0000 C CNN
+F 1 "82.5k" H 7700 2600 50  0000 C CNN
+F 2 "agg:0402" H 7650 2650 50  0001 C CNN
+F 3 "" H 7650 2650 50  0001 C CNN
+F 4 "2694663" H 200 1750 60  0001 C CNN "Farnell"
+	1    7650 2650
+	0    -1   -1   0
+$EndComp
+Wire Wire Line
+	7650 2550 7650 2200
+Wire Wire Line
+	7650 2200 8450 2200
+$Comp
+L agg-kicad1:GND #PWR0122
+U 1 1 5AE46068
+P 7650 2750
+F 0 "#PWR0122" H 7520 2790 50  0001 L CNN
+F 1 "GND" H 7650 2650 50  0000 C CNN
+F 2 "" H 7650 2750 60  0000 C CNN
+F 3 "" H 7650 2750 60  0000 C CNN
+	1    7650 2750
+	1    0    0    -1
+$EndComp
+Wire Wire Line
+	7650 2750 7650 2650
+Text Notes 5100 3650 0    60   ~ 0
+12v @ 8A Max.
+Text Notes 8500 3650 0    60   ~ 0
+12v @ 8A Max.
 $EndSCHEMATC
