File: m4dl/m4dl.sch (KiCad schematic (older format))
At the start: 38 parts, among them IC1 STM32F405RxTx, IC2 ADP3335, IC3 MCP2562, J1 WEST TOP, J2 WEST BOT, J3 EAST TOP, J4 EAST BOT, J5 NORTH TOP, P1 SWD_TC, U1 MICROSD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

Commit message: moved pwr switch and removed chg from golbal interconnect
Connections:
- net labels added: RSVD12, RSVD13
- net labels removed: CHARGE
Changed lines of the file:
@@
 5v_CAM1
 Text Label 2800 2250 2    60   ~ 0
-CHARGE
-Text Label 3300 2250 0    60   ~ 0
-CHARGE
-Text Label 3300 2150 0    60   ~ 0
 PWR
 Text Label 3300 1350 0    60   ~ 0
@@
 Wire Wire Line
 	2900 2050 2800 2050
-Wire Wire Line
-	2800 2250 2900 2250
-Wire Wire Line
-	3200 2250 3300 2250
 Wire Wire Line
 	3300 2150 3200 2150
@@
 Text Label 2800 4000 2    60   ~ 0
 5v_CAM1
-Text Label 2800 4200 2    60   ~ 0
-CHARGE
-Text Label 3300 4200 0    60   ~ 0
-CHARGE
-Text Label 3300 4100 0    60   ~ 0
-PWR
 Text Label 3300 3300 0    60   ~ 0
 PYRO4
@@
 Wire Notes Line
 	5800 5200 5800 750
+Wire Wire Line
+	2800 2250 2900 2250
+Wire Wire Line
+	3200 2250 3300 2250
+Text Label 3300 2150 0    60   ~ 0
+RSVD12
+Text Label 3300 2250 0    60   ~ 0
+RSVD13
+Text Label 2800 4200 2    60   ~ 0
+PWR
+Text Label 3300 4100 0    60   ~ 0
+RSVD12
+Text Label 3300 4200 0    60   ~ 0
+RSVD13
 $EndSCHEMATC

Commit message: strain gauge circuit added to data logger
Parts:
- added C? (x2): 8.2n, symbol strain_1-3-cache:C_Small
- added C? (x2): 82n, symbol strain_1-3-cache:C_Small
- added IC? (x2): AD8656, agg:MSOP-8, symbol strain_1-3-cache:AD8656
- added R?: 1.69K, symbol strain_1-3-cache:R
- added R?: 6.04K, symbol strain_1-3-cache:R
- added R?: 562, symbol strain_1-3-cache:R
- added R?: 17.8K, symbol strain_1-3-cache:R
- C1, C10, C11, C12, C13, C14, C15, C16, C17, C2, C3, C4, C5, C6, C7, C8, C9: symbol agg-kicad:C -> m4dl-rescue:C-agg-kicad
- D1, D2: symbol agg-kicad:LED -> m4dl-rescue:LED-agg-kicad
- IC1: symbol agg-kicad:STM32F405RxTx -> m4dl-rescue:STM32F405RxTx-agg-kicad
- IC2: symbol agg-kicad:ADP3335 -> m4dl-rescue:ADP3335-agg-kicad
- IC3: symbol agg-kicad:MCP2562 -> m4dl-rescue:MCP2562-agg-kicad
- J1, J2, J3, J4, J5: symbol agg-kicad:CONN_02x15 -> m4dl-rescue:CONN_02x15-agg-kicad
- P1: symbol agg-kicad:SWD_TC -> m4dl-rescue:SWD_TC-agg-kicad
- R1, R2, R3, R4, R5, R6, R7, R8: symbol agg-kicad:R -> m4dl-rescue:R-agg-kicad
- U1: symbol agg-kicad:MICROSD -> m4dl-rescue:MICROSD-agg-kicad
- Y1: symbol agg-kicad:SMD_XTAL -> m4dl-rescue:SMD_XTAL-agg-kicad
Connections:
- wire segments 383 -> 411

Commit message: strain gauge filter circuit added
Parts:
- R?: value 562 -> 562R
Changed lines of the file:
@@
 P 9800 1600
 F 0 "R?" V 9593 1600 50  0000 C CNN
-F 1 "562" V 9684 1600 50  0000 C CNN
+F 1 "562R" V 9684 1600 50  0000 C CNN
 F 2 "" V 9730 1600 50  0000 C CNN
 F 3 "" H 9800 1600 50  0000 C CNN

Commit message: updated pressure label, groundss
Parts:
- removed R?: 1.69K, symbol strain_1-3-cache:R
- added C19, C20, C21, C23, C24: C_Small, symbol strain_1-3-cache:C_Small
- added D3, D4: ESD_DIODE, agg:0402, symbol strain_1-3-cache:ESD_DIODE
- added IC5: AD8495, symbol ad8495:AD8495
- added P2: CONN_2, symbol m2fc-cache:CONN_2
- added R10: 1.69K, symbol strain_1-3-cache:R
- added R12, R13, R14: R, symbol strain_1-3-cache:R
- added R9: 150, symbol strain_1-3-cache:R
- gave numbers to parts that had none: 8
Connections:
- net labels added: 3v3-agg-kicad, AGND-agg-kicad
- wire segments 411 -> 448

Commit message: Thermo circuitry added
Parts:
- added C27, C30, C32: 100n, symbol strain_1-3-cache:C_Small
- added C28: 10u, symbol strain_1-3-cache:C_Small
- added C29, C31: 10n, symbol strain_1-3-cache:C_Small
- added IC6, IC?: AD8656, agg:MSOP-8, symbol strain_1-3-cache:AD8656
- added R17: 8.87K, symbol strain_1-3-cache:R
- added R18: 31.6K, symbol strain_1-3-cache:R
- added R19: 2.94K, symbol strain_1-3-cache:R
- added R20: 95.3K, symbol strain_1-3-cache:R
- added TP? (x2): TESTPAD, symbol m2fc-cache:TESTPAD
- C19, C21, C23: value C_Small -> 100n
- C20: value C_Small -> 1u
- C24: value C_Small -> 10u
- R12, R13: value R -> 1K
- R14: value R -> 1M
Connections:
- net labels added: VAA
- wire segments 448 -> 492

Commit message: added annotations to test pads
Parts:
- gave numbers to parts that had none: 3
Changed lines of the file:
@@
 	15550 3050 15550 3600
 $Comp
-L strain_1-3-cache:AD8656 IC?
-U 1 1 5BE1C325
+L strain_1-3-cache:AD8656 IC6
+U 2 1 5BE1C325
 P 15150 3600
-F 0 "IC?" H 15300 3222 50  0000 C CNN
+F 0 "IC6" H 15300 3222 50  0000 C CNN
 F 1 "AD8656" H 15300 3313 50  0000 C CNN
 F 2 "agg:MSOP-8" H 15150 3200 50  0001 L CNN
 F 3 "" H 15150 3600 50  0001 C CNN
 F 4 "1858055" H 15150 3100 50  0001 L CNN "Farnell"
-	1    15150 3600
+	2    15150 3600
 	1    0    0    1
 $EndComp
@@
 	15050 3700 15050 4050
 $Comp
-L m2fc-cache:TESTPAD TP?
+L m2fc-cache:TESTPAD TP1
 U 1 1 5BF475C5
 P 11100 3400
-F 0 "TP?" V 11129 3352 30  0000 R CNN
+F 0 "TP1" V 11129 3352 30  0000 R CNN
 F 1 "TESTPAD" H 11100 3450 60  0001 C CNN
 F 2 "" H 11100 3400 60  0000 C CNN
@@
 	15550 3600 15650 3600
 $Comp
-L m2fc-cache:TESTPAD TP?
+L m2fc-cache:TESTPAD TP2
 U 1 1 5BF851D8
 P 15650 3600
-F 0 "TP?" V 15679 3552 30  0000 R CNN
+F 0 "TP2" V 15679 3552 30  0000 R CNN
 F 1 "TESTPAD" H 15650 3650 60  0001 C CNN
 F 2 "" H 15650 3600 60  0000 C CNN

Commit message: fixed second op amp
Parts:
- removed unit 2 of IC6
- added IC?: AD8656, agg:MSOP-8, symbol strain_1-3-cache:AD8656
Connections:
- wire segments 492 -> 491
Changed lines of the file:
@@
 	1    0    0    -1
-$EndComp
-$Comp
-L m4dl-rescue:AGND-agg-kicad #PWR078
-U 1 1 5BCB3B04
-P 15250 3250
-F 0 "#PWR078" H 15120 3290 50  0001 L CNN
-F 1 "AGND-agg-kicad" H 15250 3336 50  0000 C CNN
-F 2 "" H 15250 3250 60  0001 C CNN
-F 3 "" H 15250 3250 60  0001 C CNN
-	1    15250 3250
-	-1   0    0    1
-$EndComp
-$Comp
-L m2fc-cache:VAA #PWR079
-U 1 1 5BCB3C5F
-P 15250 3800
-F 0 "#PWR079" H 15250 3650 50  0001 C CNN
-F 1 "VAA" H 15268 3973 50  0000 C CNN
-F 2 "" H 15250 3800 60  0000 C CNN
-F 3 "" H 15250 3800 60  0000 C CNN
-	1    15250 3800
-	-1   0    0    1
 $EndComp
 Wire Wire Line
@@
 Wire Wire Line
 	15550 3050 15550 3600
-$Comp
-L strain_1-3-cache:AD8656 IC6
-U 2 1 5BE1C325
-P 15150 3600
-F 0 "IC6" H 15300 3222 50  0000 C CNN
-F 1 "AD8656" H 15300 3313 50  0000 C CNN
-F 2 "agg:MSOP-8" H 15150 3200 50  0001 L CNN
-F 3 "" H 15150 3600 50  0001 C CNN
-F 4 "1858055" H 15150 3100 50  0001 L CNN "Farnell"
-	2    15150 3600
-	1    0    0    1
-$EndComp
 Connection ~ 15550 3600
 Wire Wire Line
 	15550 3600 15550 4050
-Wire Wire Line
-	15250 3250 15250 3400
 Wire Wire Line
 	15050 3500 14650 3500
@@
 	0    -1   -1   0
 $EndComp
+$Comp
+L strain_1-3-cache:AD8656 IC?
+U 2 1 5C0C8EBA
+P 15150 3600
+F 0 "IC?" H 15300 3915 50  0000 C CNN
+F 1 "AD8656" V 15300 3824 50  0000 C CNN
+F 2 "agg:MSOP-8" H 15150 3200 50  0001 L CNN
+F 3 "" H 15150 3600 50  0001 C CNN
+F 4 "1858055" H 15150 3100 50  0001 L CNN "Farnell"
+	2    15150 3600
+	1    0    0    1
+$EndComp
 $EndSCHEMATC
