File: m4psu/3v3.sch (KiCad schematic (older format))
At the start: 75 parts, among them IC5 TPS62132, IC6 LTC2975, IC7 LTC2975, Q10 PFET, Q11 NFET, Q12 PFET, Q13 NFET, Q14 PFET, Q15 NFET, Q16 PFET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

Commit message: finished psu schematic - needs review/checking
Parts:
- renumbered C19 to C21, C20 to C22, C21 to C23, C22 to C24, C23 to C25, C24 to C26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
Connections:
- wire segments 408 -> 409
