File: m4psu/5v.sch (KiCad schematic (older format))
At the start: 44 parts, among them IC8 TPS62133, IC9 LTC2975, Q21 NFET, Q22 PFET, Q23 NFET, Q24 PFET, Q25 NFET, Q26 PFET, Q27 NFET, Q28 PFET

Commit message: finished psu schematic - needs review/checking
Parts:
- renumbered C32 to C34, C33 to C35, C34 to C36, C35 to C37, C36 to C38, C37 to C39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
Connections:
- wire segments 239 -> 240
