File: m4psu/m4psu.sch (KiCad schematic (older format))
At the start: 73 parts

Commit message: added ilim resistor to pyro board
Other:
- note added: "PYRO Max 19A @ 16v"
- note added: "Probably worth doubling up the PFET and adding in a pyro_so_div\nto meausre turn on."
- note removed: "VCC 18A @ 16v"
Changed lines of the file:
@@
 JTDO
-$Comp
-L agg-kicad1:VCC #PWR?
-U 1 1 5A94CE87
-P 5500 6100
-F 0 "#PWR?" H 5500 6210 50  0001 L CNN
-F 1 "VCC" H 5500 6190 50  0000 C CNN
-F 2 "" H 5500 6100 60  0000 C CNN
-F 3 "" H 5500 6100 60  0000 C CNN
-	1    5500 6100
-	1    0    0    -1
-$EndComp
 $Comp
 L agg-kicad1:C C?
@@
 Text Notes 4550 5800 0    98   ~ 20
 Pyro Enable
-Text Notes 8850 6000 0    60   ~ 0
-VCC 18A @ 16v
+Text Notes 6700 6000 0    60   ~ 0
+PYRO Max 19A @ 16v
 $Comp
 L agg-kicad1:PFET_GDS Q?
@@
 	-1   0    0    -1
 $EndComp
+Text Notes 4550 8100 0    60   ~ 0
+Probably worth doubling up the PFET and adding in a pyro_so_div\nto meausre turn on.
+$Comp
+L agg-kicad1:VBATT #PWR?
+U 1 1 5AFB37A7
+P 5500 6100
+F 0 "#PWR?" H 5500 6210 50  0001 L CNN
+F 1 "VBATT" H 5500 6190 50  0000 C CNN
+F 2 "" H 5500 6100 60  0000 C CNN
+F 3 "" H 5500 6100 60  0000 C CNN
+	1    5500 6100
+	1    0    0    -1
+$EndComp
 $EndSCHEMATC

Commit message: did dcdc converters
Parts:
- removed C? (x2): 2µ2, agg:0402, symbol agg-kicad1:C
- removed C? (x2): 10p, agg:0402, symbol agg-kicad1:C
- removed C? (x5): 100n, agg:0402, symbol agg-kicad1:C
- removed C?: 1µ, agg:0402, symbol agg-kicad1:C
- removed C?: 4µ7, agg:0402, symbol agg-kicad1:C
- removed C?: 100n, agg:0603, symbol agg-kicad1:C
- removed IC?: STM32F405RxTx, agg:LQFP-64, symbol agg-kicad1:STM32F405RxTx
- removed IC?: LTC4151, agg:DFN-10-EP-LT, symbol agg-kicad1:LTC4151
- removed J?: NORTH TOP, agg:TFML-105-02-L-D, symbol agg-kicad1:CONN_02x05
- removed Q?: NFET, agg:SOT-883-B, symbol agg-kicad1:NFET_GDS
- removed Q?: PFET, agg:PowerPAK-SO-8, symbol agg-kicad1:PFET_GDS
- removed R?: 100, agg:0402, symbol agg-kicad1:R
- removed R? (x3): 4k7, agg:0402, symbol agg-kicad1:R
- removed R? (x2): 33k, agg:0402, symbol agg-kicad1:R
- removed R?: 2m, agg:1206, symbol agg-kicad1:R
- removed Y?: 26M, agg:XTAL-20x16, symbol agg-kicad1:SMD_XTAL
- added C18: 100n, agg:0603, symbol agg-kicad1:C
- added IC4: LTC4151, agg:DFN-10-EP-LT, symbol agg-kicad1:LTC4151
- added Q1, Q2, Q3: PFET, agg:PowerPAK-SO-8, symbol agg-kicad1:PFET_GDS
- added Q4: NFET, agg:SOT-883-B, symbol agg-kicad1:NFET_GDS
- added R10: 2m, agg:1206, symbol agg-kicad1:R
- added R11, R12: 33k, agg:0402, symbol agg-kicad1:R
- added TP1, TP2, TP3, TP4: TESTPAD, agg:TESTPAD, symbol agg-kicad1:TESTPAD
- gave numbers to parts that had none: 48
Connections:
- net labels removed: JTDO, V_MAIN
- wire segments 443 -> 372
- no-connect marks 43 -> 4
Other:
- note added: "(VMAIN)"
- note added: "DC-DC Converters"
- note added: "Soft Power Switch"
- note removed: "PB4 is JTRST, NC (Errata 2.1.4)"
- note removed: "Probably worth doubling up the PFET and adding in a pyro_so_div\nto meausre turn on."

Commit message: finished psu schematic - needs review/checking
Parts:
- added C19, C20: 100n, agg:0603, symbol agg-kicad1:C
- added IC5: TLV76012, agg:SOT-23, symbol agg-kicad:TLV76012
- added R108: 120, agg:0603, symbol agg-kicad:R
- added R11, R15: 47k, agg:0402, symbol agg-kicad1:R
- added R12, R16: 10k, agg:0402, symbol agg-kicad1:R
- renumbered R11 to R13, R12 to R14, R13 to R17, R14 to R18
Connections:
- net labels added: 12v_DIV, SO_DIV
- wire segments 372 -> 408
- no-connect marks 4 -> 58
Other:
- note added: "12v DL Regulator"
- note added: "Charger"
- note added: "Voltage Monitoring"
- note removed: "Battery Taps"
